Commit message: task3c_resource_added

File: ros_task_2/mini_bot/urdf/mini_bot_1.urdf.xacro (robot description, xacro)
@@ -62,5 +62,5 @@
         <inertial>
             <origin
-                xyz="0 -0.05 0.0"
+                xyz="0.0 -0.05 0.0"
                 rpy="1.57 0 0" />
             <mass
@@ -76,5 +76,5 @@
          <collision name="L_collision">
          <origin
-                xyz="0 -0.05 0.0"
+                xyz="0.0 -0.05 0.0"
                 rpy="1.57 0 0" />
           <geometry>
@@ -126,9 +126,43 @@
     </link>
     <gazebo reference="Right_wheel"><material>Gazebo/Blue</material></gazebo>
+    <!-- rear_wheel -->
+    <link name ="Rear_wheel">
+        <inertial>
+            <origin
+                xyz="0.0 -0.05 0.0"
+                rpy="1.57 0.0 0.0"/>
+            <mass
+                value="0.060" />
+            <inertia
+                ixx="1.825e-4"
+                ixy="0"
+                ixz="0.00000000"
+                iyy="1.825e-4"
+                iyz="0"
+                izz="1.825e-4" />
+        </inertial>
+        <collision name="R_collision">
+        <origin
+                xyz="0.0 -0.05 0.0"
+                rpy="1.57 0.0 0.0" />
+          <geometry>
+            <cylinder length="0.13" radius="0.14"/>
+          </geometry>
+        </collision>
+        <visual>
+            <origin
+            xyz="0.0 0.0 0.0"
+            rpy="0 0 0.0" />
+            <geometry>
+                <mesh filename ="file://$(find mini_bot)/meshes/wheel.stl" scale="5 5 5"/>
+            </geometry>
+        </visual>
+    </link>
+    <gazebo reference="Rear_wheel"><material>Gazebo/Green</material></gazebo>
    <!-- joints -->
     <!--Right wheel joint -->
     <joint name ="Right_wheel_joint" type="continuous" >
         <origin
-             xyz="0.58 -0.36 0.18"
+            xyz="0.58 -0.36 0.18"
             rpy="0.0 0.0 -2.12" />
         <parent link="base_link"/>
@@ -142,6 +176,6 @@
     <joint name ="Left_wheel_joint" type="continuous" >
         <origin
-                xyz="0.0 0.68 0.18"
-                rpy="0 0 0" />
+            xyz="0.0 0.68 0.18"
+            rpy="0 0 0" />
         <parent link="base_link"/>
         <child link="Left_wheel"/>
@@ -151,4 +185,27 @@
             velocity="5" />
     </joint>
+    <!-- Joint -->
+    <!--Rear wheel joint -->
+    <joint name ="Rear_wheel_joint" type="continuous" >
+        <origin
+            xyz="-0.58 -0.32 0.18"
+            rpy="0.0 0.0 2.12" />
+        <parent link="base_link"/>
+        <child link="Rear_wheel"/>
+        <axis xyz="0.0 1.0 0.0"/>
+         <limit
+            effort="5"
+            velocity="5" />
+    </joint>
     <!-- plug-ins -->
+    <gazebo>
+      <plugin name="planar_move" filename="libgazebo_ros_planar_move.so">
+        <commandTopic>cmd_vel</commandTopic>
+        <odometryTopic>odom</odometryTopic>
+        <odometryFrame>odom</odometryFrame>
+        <robotBaseFrame>base_link</robotBaseFrame>
+        <odometryRate>100</odometryRate>
+        <enableMotors>true</enableMotors>
+     </plugin>
+   </gazebo>
 </robot>
